File: PCB-Files/Keyboard.kicad_pcb (KiCad board)
At the start: 2 copper layers, 342.1 x 123 mm, 167 parts

Commit message: Updating the PCB design
I updated the PCB design this should hopefully fix some of the issues I was having
Other:
- board text removed: "Created by Fastturtle25 Thank you to Hackclub and Keeb for making this possible"
- board text removed: "Ortho-Turtle"
Changed lines of the file:
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@@
 			(outputformat 1)
 			(mirror no)
-			(drillshape 0)
+			(drillshape 1)
 			(scaleselection 1)
-			(outputdirectory "C:/Users/Jackson/Documents/OrthoTurtle-PCB-files/")
+			(outputdirectory "")
 		)
 	)
@@
 		(layer "Edge.Cuts")
 	)
-	(gr_text "Created by Fastturtle25\nThank you to Hackclub and Keeb for making this possible"
-		(at 380.1823 136.5164 90)
-		(layer "F.SilkS")
-		(effects
-			(font
-				(size 1 1)
-				(thickness 0.1)
-			)
-			(justify left bottom)
-		)
-	)
-	(gr_text "Ortho-Turtle"
-		(at 69.8456 94.4503 0)
-		(layer "F.SilkS")
-		(effects
-			(font
-				(size 25 25)
-				(thickness 5)
-				(bold yes)
-				(italic yes)
-			)
-			(justify left bottom)
-		)
-	)
 	(segment
 		(start 84.9259 39.0165)
@@
 	)
 	(segment
-		(start 51.06 33.02)
-		(end 51.1122 33.02)
-		(width 0.2)
-		(layer "F.Cu")
-		(net "Net-(D1-A)")
-	)
-	(segment

Commit message: Final PCB fixes
These should be the final fixes for the PCB including fixing the Pi picos grounding and doing logos
Routing:
- added copper zone on F.Cu, net Net-(A1-GND-Pad13)
Other:
- board text added: "Created by Fastturtle25 Thank you to Hackclub and Keeb for making this possible"
- board text added: "Ortho-Turtle"
Changed lines of the file:
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@@
 			(outputformat 1)
 			(mirror no)
-			(drillshape 1)
+			(drillshape 0)
 			(scaleselection 1)
-			(outputdirectory "")
+			(outputdirectory "C:/Users/Jackson/Documents/OrthoTurtle-PCB-files/")
 		)
 	)
@@
 		(layer "Edge.Cuts")
 	)
+	(gr_text "Created by Fastturtle25\nThank you to Hackclub and Keeb for making this possible"
+		(at 380.1823 136.5164 90)
+		(layer "F.SilkS")
+		(effects
+			(font
+				(size 1 1)
+				(thickness 0.1)
+			)
+			(justify left bottom)
+		)
+	)
+	(gr_text "Ortho-Turtle"
+		(at 69.8456 94.4503 0)
+		(layer "F.SilkS")
+		(effects
+			(font
+				(size 25 25)
+				(thickness 5)
+				(bold yes)
+				(italic yes)
+			)
+			(justify left bottom)
+		)
+	)
 	(segment
 		(start 84.9259 39.0165)
@@
 		(net "Net-(D2-A)")
 	)
+	(zone
+		(net "Net-(A1-GND-Pad13)")
+		(layer "F.Cu")
+		(hatch edge 0.5)
+		(connect_pads
+			(clearance 0.5)
+		)
+		(min_thickness 0.25)
+		(fill yes
+			(thermal_gap 0.5)
+			(thermal_bridge_width 0.5)
+			(island_removal_mode 0)
+		)
+		(polygon
+			(pts
+				(xy -8.7307 -7.937) (xy -13.4929 163.5022) (xy 439.7098 176.2014) (xy 443.6783 -37.3039) (xy -11.1118 -9.5244)
+			)
+		)
+	)
 	(embedded_fonts no)
